Commit message: Camera

File: src/my_r2d2/urdf/r2d2.urdf.xacro (robot description, xacro)
@@ -225,3 +225,15 @@
     <origin xyz="0 0 ${bodylen/2+wheeldiam+0.1}" rpy="0 0 0"/>
   </joint>
+  <link name="eye">
+    <visual>
+      <geometry>
+        <cylinder/>
+      </geometry>
+    </visual>
+  </link>
+  <joint name="eye_joint" type="fixed">
+    <parent link="box"/>
+    <child link="eye"/>
+    <origin xyz="-0.04 0 0" rpy="${pi/2} ${pi} ${pi/2}"/>
+  </joint>
 </robot>
